Commit message: fixed lane

File: src/main_bot/description/lidar.xacro (robot description, xacro)
@@ -26,5 +26,5 @@
     <parent link="base_link"/>
     <child  link="lidar_frame"/>
-    <origin xyz="0 0 ${chassis_height/2 + lidar_height/2}" rpy="0 0 0"/>
+    <origin xyz="0 0 ${chassis_height/2 + lidar_height/2 + 0.03}" rpy="0 0 0"/>
   </joint>
   <!-- ─── Gazebo sensor ─── -->

File: src/main_bot/description/robot.urdf.xacro (robot description, xacro)
@@ -5,3 +5,4 @@
     <xacro:include filename="lidar.xacro"/>
     <xacro:include filename="camera.xacro"/>
+    <xacro:include filename="imu.xacro"/>
 </robot>
